Commit message: Configure for 2 dynamixels

File: tests/test_joint.xacro (robot description, xacro)
@@ -12,5 +12,5 @@
   <xacro:include filename="$(find dynamixel_ros_control)/tests/materials.xacro" />
   <!-- Base Link -->
-  <link name="link1">
+  <link name="link_base">
     <collision>
       <origin xyz="0 0 ${height1/2}" rpy="0 0 0"/>
@@ -36,6 +36,6 @@
   </link>
   <joint name="joint1" type="continuous">
-    <parent link="link1"/>
-    <child link="link2"/>
+    <parent link="link_base"/>
+    <child link="link1"/>
     <origin xyz="0 ${width} ${height1 - axel_offset}" rpy="0 0 0"/>
     <axis xyz="0 1 0"/>
@@ -43,5 +43,5 @@
   </joint>
   <!-- Middle Link -->
-  <link name="link2">
+  <link name="link1">
     <collision>
       <origin xyz="0 0 ${height2/2 - axel_offset}" rpy="0 0 0"/>
@@ -66,4 +66,35 @@
     </inertial>
   </link>
+  <joint name="joint2" type="continuous">
+    <parent link="link_base"/>
+    <child link="link2"/>
+    <origin xyz="0 ${width} ${height1 - axel_offset}" rpy="0 0 0"/>
+    <axis xyz="0 1 0"/>
+    <dynamics damping="0.7"/>
+  </joint>
+  <!-- Middle Link -->
+  <link name="link2">
+    <collision>
+      <origin xyz="0 0 ${height2/2 - axel_offset}" rpy="0 0 0"/>
+      <geometry>
+  <box size="${width} ${width} ${height2}"/>
+      </geometry>
+    </collision>
+    <visual>
+      <origin xyz="0 0 ${height2/2 - axel_offset}" rpy="0 0 0"/>
+      <geometry>
+  <box size="${width} ${width} ${height2}"/>
+      </geometry>
+      <material name="black"/>
+    </visual>
+    <inertial>
+      <origin xyz="0 0 ${height2/2 - axel_offset}" rpy="0 0 0"/>
+      <mass value="${mass}"/>
+      <inertia
+    ixx="${mass / 12.0 * (width*width + height2*height2)}" ixy="0.0" ixz="0.0"
+    iyy="${mass / 12.0 * (height2*height2 + width*width)}" iyz="0.0"
+    izz="${mass / 12.0 * (width*width + width*width)}"/>
+    </inertial>
+  </link>
   <transmission name="tran1">
     <type>transmission_interface/SimpleTransmission</type>

Commit message: Create a gripper in urdf

File: tests/test_joint.xacro (robot description, xacro)
@@ -2,11 +2,9 @@
 <robot name="test_joint" xmlns:xacro="http://www.ros.org/wiki/xacro">
   <xacro:property name="PI" value="3.1415926535897931"/>
-  <xacro:property name="mass" value="1" /> <!-- arbitrary value for mass -->
-  <xacro:property name="width" value="0.1" /> <!-- Square dimensions (widthxwidth) of beams -->
-  <xacro:property name="height1" value="2" /> <!-- Link 1 -->
-  <xacro:property name="height2" value="1" /> <!-- Link 2 -->
-  <xacro:property name="height3" value="1" /> <!-- Link 3 -->
-  <xacro:property name="camera_link" value="0.05" /> <!-- Size of square 'camera' box -->
-  <xacro:property name="axel_offset" value="0.05" /> <!-- Space btw top of beam and the each joint -->
+  <xacro:property name="base_width" value="0.08" />
+  <xacro:property name="base_height" value="0.06" />
+  <xacro:property name="base_depth" value="0.03" />
+  <xacro:property name="gripper_width" value="0.02" />
+  <xacro:property name="gripper_height" value="0.1" />
   <!-- Import Rviz colors -->
   <xacro:include filename="$(find dynamixel_ros_control)/tests/materials.xacro" />
@@ -14,86 +12,39 @@
   <link name="link_base">
     <collision>
-      <origin xyz="0 0 ${height1/2}" rpy="0 0 0"/>
+      <origin xyz="0 0 ${base_height/2}" rpy="0 0 0"/>
       <geometry>
-	<box size="${width} ${width} ${height1}"/>
+	      <box size="${base_width} ${base_depth} ${base_height}"/>
       </geometry>
     </collision>
     <visual>
-      <origin xyz="0 0 ${height1/2}" rpy="0 0 0"/>
+      <origin xyz="0 0 ${base_height/2}" rpy="0 0 0"/>
       <geometry>
-	<box size="${width} ${width} ${height1}"/>
+	      <box size="${base_width} ${base_depth} ${base_height}"/>
       </geometry>
       <material name="orange"/>
     </visual>
-    <inertial>
-      <origin xyz="0 0 ${height1/2}" rpy="0 0 0"/>
-      <mass value="${mass}"/>
-      <inertia
-	  ixx="${mass / 12.0 * (width*width + height1*height1)}" ixy="0.0" ixz="0.0"
-	  iyy="${mass / 12.0 * (height1*height1 + width*width)}" iyz="0.0"
-	  izz="${mass / 12.0 * (width*width + width*width)}"/>
-    </inertial>
   </link>
-  <joint name="joint1" type="continuous">
+  <joint name="joint1" type="revolute">
     <parent link="link_base"/>
     <child link="link1"/>
-    <origin xyz="0 ${width} ${height1 - axel_offset}" rpy="0 0 0"/>
+    <origin xyz="${base_width/2} 0 ${base_height}" rpy="0 0 0"/>
     <axis xyz="0 1 0"/>
-    <dynamics damping="0.7"/>
+    <limit lower="-0.35" upper="${PI/2}" effort="1" velocity="1" />
   </joint>
   <!-- Middle Link -->
   <link name="link1">
     <collision>
-      <origin xyz="0 0 ${height2/2 - axel_offset}" rpy="0 0 0"/>
+      <origin xyz="0 0 ${gripper_height/2}" rpy="0 0 0"/>
       <geometry>
-	<box size="${width} ${width} ${height2}"/>
+	      <box size="${gripper_width} ${gripper_width} ${gripper_height}"/>
       </geometry>
     </collision>
     <visual>
-      <origin xyz="0 0 ${height2/2 - axel_offset}" rpy="0 0 0"/>
+      <origin xyz="0 0 ${gripper_height/2}" rpy="0 0 0"/>
       <geometry>
-	<box size="${width} ${width} ${height2}"/>
+        <box size="${gripper_width} ${gripper_width} ${gripper_height}"/>
       </geometry>
       <material name="black"/>
     </visual>
-    <inertial>
-      <origin xyz="0 0 ${height2/2 - axel_offset}" rpy="0 0 0"/>
-      <mass value="${mass}"/>
-      <inertia
-	  ixx="${mass / 12.0 * (width*width + height2*height2)}" ixy="0.0" ixz="0.0"
-	  iyy="${mass / 12.0 * (height2*height2 + width*width)}" iyz="0.0"
-	  izz="${mass / 12.0 * (width*width + width*width)}"/>
-    </inertial>
-  </link>
-  <joint name="joint2" type="continuous">
-    <parent link="link_base"/>
-    <child link="link2"/>
-    <origin xyz="0 ${width} ${height1 - axel_offset}" rpy="0 0 0"/>
-    <axis xyz="0 1 0"/>
-    <dynamics damping="0.7"/>
-  </joint>
-  <!-- Middle Link -->
-  <link name="link2">
-    <collision>
-      <origin xyz="0 0 ${height2/2 - axel_offset}" rpy="0 0 0"/>
-      <geometry>
-  <box size="${width} ${width} ${height2}"/>
-      </geometry>
-    </collision>
-    <visual>
-      <origin xyz="0 0 ${height2/2 - axel_offset}" rpy="0 0 0"/>
-      <geometry>
-  <box size="${width} ${width} ${height2}"/>
-      </geometry>
-      <material name="black"/>
-    </visual>
-    <inertial>
-      <origin xyz="0 0 ${height2/2 - axel_offset}" rpy="0 0 0"/>
-      <mass value="${mass}"/>
-      <inertia
-    ixx="${mass / 12.0 * (width*width + height2*height2)}" ixy="0.0" ixz="0.0"
-    iyy="${mass / 12.0 * (height2*height2 + width*width)}" iyz="0.0"
-    izz="${mass / 12.0 * (width*width + width*width)}"/>
-    </inertial>
   </link>
   <transmission name="tran1">
